Commit message: added cam link and joint but does not show in gazebo

File: mybot_description/urdf/mybot.xacro (robot description, xacro)
@@ -95,4 +95,24 @@
     </inertial>
   </link>
+   <!-- Sensor links -->
+  <link name="cam_link">
+    <collision name="cam_collision">
+      <origin xyz="0 0 0" rpy="0 0 0"/>
+      <geometry>
+        <box size="0.05 0.05 0.05"/>
+      </geometry>
+    </collision>
+    <visual name="cam_vis">
+      <origin xyz="0 0 0" rpy="0 0 0"/>
+      <geometry>
+        <box size="0.05 0.05 0.05"/>
+      </geometry>
+    </visual>
+    <inertial>
+      <mass value="1e-5" />
+      <origin xyz="0 0 0" rpy="0 0 0"/>
+      <inertia ixx="1e-6" ixy="0" ixz="0" iyy="1e-6" iyz="0" izz="1e-6" />
+    </inertial>
+  </link>
   <joint type="continuous" name="left_wheel_hinge">
     <origin xyz="0.07 0.09 -0.02" rpy="0 0 0"/>
@@ -111,3 +131,9 @@
     <joint_properties damping="0.0" friction="0.0"/>
   </joint>
+  <joint type="fixed" name="cam_joint">
+    <axis xyz="0 0 1" />
+    <origin xyz="-0.12 0 0.13" rpy="0 0 0"/>
+    <parent link="chassis"/>
+    <child link="cam_link"/>
+  </joint>
 </robot>

Commit message: Tried adding link and joint for camera

File: mybot_description/urdf/mybot.xacro (robot description, xacro)
@@ -19,8 +19,8 @@
     </collision>
     <visual name='chassis_visual'>
-              <origin xyz="0 0 0.03" rpy="0.0 0.0 1.57" />
-        <geometry>
-          <mesh filename="package://mybot_description/meshes/frobit_base.stl" />
-        </geometry>
+      <origin xyz="0 0 0.03" rpy="0.0 0.0 1.57" />
+      <geometry>
+        <mesh filename="package://mybot_description/meshes/frobit_base.stl" />
+      </geometry>
     </visual>
     <collision name='caster_collision'>
@@ -109,9 +109,4 @@
       </geometry>
     </visual>
-    <inertial>
-      <mass value="1e-5" />
-      <origin xyz="0 0 0" rpy="0 0 0"/>
-      <inertia ixx="1e-6" ixy="0" ixz="0" iyy="1e-6" iyz="0" izz="1e-6" />
-    </inertial>
   </link>
   <joint type="continuous" name="left_wheel_hinge">
@@ -132,8 +127,8 @@
   </joint>
   <joint type="fixed" name="cam_joint">
+    <origin xyz="0 -0.10 0.07" rpy="0 0 0"/>
+    <child link="cam_link"/>
+    <parent link="chassis"/>
     <axis xyz="0 0 1" />
-    <origin xyz="-0.12 0 0.13" rpy="0 0 0"/>
-    <parent link="chassis"/>
-    <child link="cam_link"/>
   </joint>
 </robot>

Commit message: Cam sensor working

File: mybot_description/urdf/mybot.xacro (robot description, xacro)
@@ -127,8 +127,8 @@
   </joint>
   <joint type="fixed" name="cam_joint">
-    <origin xyz="0 -0.10 0.07" rpy="0 0 0"/>
+    <origin xyz="0 -0.10 0.07" rpy="0 0 -1.5707"/>
     <child link="cam_link"/>
     <parent link="chassis"/>
-    <axis xyz="0 0 1" />
+    <axis xyz="0 0 0" />
   </joint>
 </robot>
