Commit message: Init branch

File: simulation/mybot_description/urdf/mybot.xacro (robot description, xacro)
@@ -104,9 +104,23 @@
     </collision>
     <visual name="cam_vis">
-      <origin xyz="0 0 0" rpy="0 0 0"/>
+      <origin xyz="0 0 0.028" rpy="0 0 -1.5707"/>
       <geometry>
-        <box size="0.05 0.05 0.05"/>
+        <mesh filename="package://mybot_description/meshes/sport_camera.dae"/>
       </geometry>
     </visual>
+  </link>
+  <link name="gps_link">
+    <visual>
+      <origin xyz="0 0 0" rpy="0 0 0" />
+      <geometry>
+        <box size="0.01 0.01 0.01" />
+      </geometry>
+    </visual>
+    <collision>
+      <origin xyz="0 0 0" rpy="0 0 0" />
+      <geometry>
+        <box size="0.01 0.01 0.01" />
+      </geometry>
+    </collision>
   </link>
   <joint type="continuous" name="left_wheel_hinge">
@@ -126,4 +140,5 @@
     <joint_properties damping="0.0" friction="0.0"/>
   </joint>
+  <!-- Sensor joints -->
   <joint type="fixed" name="cam_joint">
     <origin xyz="0 -0.10 0.07" rpy="0 0 -1.5707"/>
@@ -132,3 +147,8 @@
     <axis xyz="0 0 0" />
   </joint>
+  <joint name="gps_joint" type="fixed">
+    <origin xyz="0 0 0.07"/>
+    <parent link="chassis"/>
+    <child link="gps_link"/>
+  </joint>
 </robot>

Commit message: chaanged the orientation and implemented Lidar

File: simulation/mybot_description/urdf/mybot.xacro (robot description, xacro)
@@ -4,9 +4,15 @@
   <xacro:include filename="$(find mybot_description)/urdf/materials.xacro" />
   <xacro:include filename="$(find mybot_description)/urdf/macros.xacro" />
+<!--<link name='base_link'/>
+<joint type="fixed" name="world_to_chassis_joint">
+<origin xyz="0 0 0" rpy="0 0 0"/>
+<parent link="base_link"/>
+<child link="chassis"/>
+</joint>-->
   <link name='chassis'>
-    <pose>0 0 0.1 0 0 0</pose>
+    <pose>0 0 0.1 0 0 </pose>
     <inertial>
-      <mass value="3.0"/>
-      <origin xyz="0.0 0 0.1" rpy=" 0 0 0"/>
+      <mass value="10.0"/>
+      <origin xyz="0.0 0 0.06" rpy=" 0 0 0"/>
       <inertia ixx="0.021318375" ixy="0"  ixz="0"
              iyy="0.030650708" iyz="-0.000002"
@@ -14,4 +20,5 @@
       </inertial>
     <collision name='collision'>
+<origin xyz="0.0 0.0 0.0" rpy=" 0 0 0"/>
       <geometry>
         <box size=".4 .2 .1"/>
@@ -19,11 +26,11 @@
     </collision>
     <visual name='chassis_visual'>
-      <origin xyz="0 0 0.03" rpy="0.0 0.0 1.57" />
-      <geometry>
-        <mesh filename="package://mybot_description/meshes/frobit_base.stl" />
-      </geometry>
+          <origin xyz="0 0 0.06" rpy="0.0 0.0 -1.57" />
+        <geometry>
+          <mesh filename="package://mybot_description/meshes/frobit_base.stl" />
+        </geometry>
     </visual>
-    <collision name='caster_collision'>
-      <origin xyz="-0.15 0 -0.05" rpy=" 0 0 0"/>
+  <!--  <collision name='caster_collision'>
+      <origin xyz="-0.15 0 0.05" rpy=" 0 0 0"/>
       <geometry>
         <sphere radius="0.03"/>
@@ -34,6 +41,6 @@
             <mu>0</mu>
             <mu2>0</mu2>
-            <slip1>1.0</slip1>
-            <slip2>1.0</slip2>
+            <slip1>0.0</slip1>
+            <slip2>0.0</slip2>
           </ode>
         </friction>
@@ -41,14 +48,41 @@
     </collision>
     <visual name='caster_visual'>
-      <origin xyz="-0.15 0 0.04" rpy=" 0 0 1.57"/>
+      <origin xyz="0.15 0 0.06" rpy=" 0 0 -1.57"/>
+      <geometry>
+        <mesh filename="package://mybot_description/meshes/front_wheel.stl" />
+      </geometry>
+    </visual>-->
+  </link>
+<joint name="caster_joint" type="fixed">
+            <parent link="chassis"/>
+            <child link="caster_link"/>
+      </joint>
+<link name="caster_link">
+    <collision name="collision">
+      <origin xyz="0.15 0 0.06" rpy=" 0 0 0"/>
+      <geometry>
+        <cylinder radius="0.05" length="0.04"/>
+      </geometry>
+    </collision>
+    <visual name="caster_visual">
+      <origin xyz="0.15 0 0.06" rpy=" 0 0 -1.57"/>
       <geometry>
         <mesh filename="package://mybot_description/meshes/front_wheel.stl" />
       </geometry>
     </visual>
+<inertial>
+      <origin xyz="0 0 0.0" rpy="0 1.5707 1.5707"/>
+      <mass value="1"/>
+      <cylinder_inertia m="1" r="0.05" h="0.04"/>
+      <inertia
+        ixx="1.0" ixy="0.0" ixz="0.0"
+        iyy="1.0" iyz="0.0"
+        izz="1.0"/>
+    </inertial>
   </link>
   <link name="left_wheel">
     <!--origin xyz="0.1 0.13 0.1" rpy="0 1.5707 1.5707"/-->
     <collision name="collision">
-      <origin xyz="0 0 0" rpy="0 1.5707 1.5707"/>
+      <origin xyz="0 0 0.0" rpy="0 1.5707 1.5707"/>
       <geometry>
         <cylinder radius="0.05" length="0.04"/>
@@ -56,5 +90,5 @@
     </collision>
     <visual name="left_wheel_visual">
-      <origin xyz="0 0 0" rpy="1.57 0 1.57"/>
+      <origin xyz="0 0 0.0" rpy="1.57 0 1.57"/>
       <geometry>
         <mesh filename="package://mybot_description/meshes/frobit_wheel.stl" />
@@ -62,5 +96,5 @@
     </visual>
     <inertial>
-      <origin xyz="0 0 0" rpy="0 1.5707 1.5707"/>
+      <origin xyz="0 0 0.0" rpy="0 1.5707 1.5707"/>
       <mass value="5"/>
       <cylinder_inertia m="5" r="0.05" h="0.04"/>
@@ -74,5 +108,5 @@
     <!--origin xyz="0.1 -0.13 0.1" rpy="0 1.5707 1.5707"/-->
     <collision name="collision">
-      <origin xyz="0 0 0" rpy="0 1.5707 1.5707"/>
+      <origin xyz="0 0 0.0" rpy="0 1.5707 1.5707"/>
       <geometry>
         <cylinder radius="0.05" length="0.04"/>
@@ -80,5 +114,5 @@
     </collision>
     <visual name="right_wheel_visual">
-      <origin xyz="0 0 0" rpy="1.57 0 -1.57"/>
+      <origin xyz="0 0 0.0" rpy="1.57 0 -1.57"/>
       <geometry>
         <mesh filename="package://mybot_description/meshes/frobit_wheel.stl" />
@@ -86,5 +120,5 @@
     </visual>
     <inertial>
-      <origin xyz="0 0 0" rpy="0 1.5707 1.5707"/>
+      <origin xyz="0 0 0.0" rpy="0 1.5707 1.5707"/>
       <mass value="5"/>
       <cylinder_inertia m="5" r="0.05" h="0.04"/>
@@ -95,40 +129,46 @@
     </inertial>
   </link>
-   <!-- Sensor links -->
-  <link name="cam_link">
-    <collision name="cam_collision">
-      <origin xyz="0 0 0" rpy="0 0 0"/>
-      <geometry>
-        <box size="0.05 0.05 0.05"/>
-      </geometry>
-    </collision>
-    <visual name="cam_vis">
-      <origin xyz="0 0 0" rpy="0 0 0"/>
-      <geometry>
-        <box size="0.05 0.05 0.05"/>
-      </geometry>
-    </visual>
-  </link>
   <joint type="continuous" name="left_wheel_hinge">
-    <origin xyz="0.07 0.09 -0.02" rpy="0 0 0"/>
+    <origin xyz="-0.07 0.09 0" rpy="0 0 0"/>
+    <parent link="chassis"/>
     <child link="left_wheel"/>
-    <parent link="chassis"/>
     <axis xyz="0 1 0" rpy="0 0 0"/>
     <limit effort="100" velocity="100"/>
-    <joint_properties damping="0.0" friction="0.0"/>
+    <joint_properties damping="1.0" friction="0.1"/>
   </joint>
   <joint type="continuous" name="right_wheel_hinge">
-    <origin xyz="0.07 -0.09 -0.02" rpy="0 0 0"/>
+    <origin xyz="-0.07 -0.09 0" rpy="0 0 0"/>
+    <parent link="chassis"/>
     <child link="right_wheel"/>
-    <parent link="chassis"/>
     <axis xyz="0 1 0" rpy="0 0 0"/>
     <limit effort="100" velocity="100"/>
-    <joint_properties damping="0.0" friction="0.0"/>
+    <joint_properties damping="1.0" friction="0.1"/>
   </joint>
-  <joint type="fixed" name="cam_joint">
-    <origin xyz="0 -0.10 0.07" rpy="0 0 -1.5707"/>
-    <child link="cam_link"/>
-    <parent link="chassis"/>
-    <axis xyz="0 0 0" />
+ <joint name="laser_joint" type="fixed">
+    <origin xyz="0.17 0 0.1" rpy="0 0 3.1416" />
+    <parent link="chassis" />
+    <child link="laser" />
   </joint>
+<!--
+ <joint name="front_wheel_joint" type="revolute">
+    <origin xyz="0.17 0 0.1" rpy="0 0 3.1416" />
+    <parent link="chassis" />
+    <child link="laser" />
+  </joint>
+-->
+<link name="laser">
+	<visual>
+	<geometry>
+	<mesh filename="package://mybot_description/meshes/hokuyo.dae" />
+ 	</geometry>
+	<material name="Green"/>
+	</visual>
+	<inertial>
+ 	<mass value="0.001"/>
+	<inertia
+	ixx="0.0001" ixy="0.0" ixz="0.0"
+	iyy="0.0001" iyz="0.0"
+ 	izz="0.0001"/>
+ 	</inertial>
+ </link>
 </robot>

Commit message: Done with GPS node

File: simulation/mybot_description/urdf/mybot.xacro (robot description, xacro)
@@ -148,5 +148,5 @@
   </joint>
   <joint name="gps_joint" type="fixed">
-    <origin xyz="0 0 0.07"/>
+    <origin xyz="0 0.5 0.07"/>
     <parent link="chassis"/>
     <child link="gps_link"/>

Commit message: added so image and metadata can be saved

File: simulation/mybot_description/urdf/mybot.xacro (robot description, xacro)
@@ -145,10 +145,10 @@
   </link>
   <link name="laser">
-	  <visual>
-	    <geometry>
-	      <mesh filename="package://mybot_description/meshes/hokuyo.dae" />
- 	    </geometry>
-	    <material name="Green"/>
-	  </visual>
+    <visual>
+      <geometry>
+        <mesh filename="package://mybot_description/meshes/hokuyo.dae" />
+      </geometry>
+      <material name="Green"/>
+    </visual>
   </link>
   <link name="gps_link">

Commit message: trying to correct bug with roslaunch

File: simulation/mybot_description/urdf/mybot.xacro (robot description, xacro)
@@ -20,5 +20,5 @@
       </inertial>
     <collision name='collision'>
-<origin xyz="0.0 0.0 0.0" rpy=" 0 0 0"/>
+      <origin xyz="0.0 0.0 0.0" rpy=" 0 0 0"/>
       <geometry>
         <box size=".4 .2 .1"/>
@@ -26,5 +26,5 @@
     </collision>
     <visual name='chassis_visual'>
-          <origin xyz="0 0 0.06" rpy="0.0 0.0 -1.57" />
+        <origin xyz="0 0 0.06" rpy="0.0 0.0 -1.57" />
         <geometry>
           <mesh filename="package://mybot_description/meshes/frobit_base.stl" />
@@ -54,29 +54,29 @@
     </visual>-->
   </link>
-<joint name="caster_joint" type="fixed">
-            <parent link="chassis"/>
-            <child link="caster_link"/>
-      </joint>
-<link name="caster_link">
+  <joint name="caster_joint" type="fixed">
+    <parent link="chassis"/>
+    <child link="caster_link"/>
+  </joint>
+  <link name="caster_link">
     <collision name="collision">
       <origin xyz="0.15 0 0.06" rpy=" 0 0 0"/>
-      <geometry>
-        <cylinder radius="0.05" length="0.04"/>
-      </geometry>
+        <geometry>
+          <cylinder radius="0.05" length="0.04"/>
+        </geometry>
     </collision>
     <visual name="caster_visual">
       <origin xyz="0.15 0 0.06" rpy=" 0 0 -1.57"/>
-      <geometry>
-        <mesh filename="package://mybot_description/meshes/front_wheel.stl" />
-      </geometry>
-    </visual>
-<inertial>
-      <origin xyz="0 0 0.0" rpy="0 1.5707 1.5707"/>
-      <mass value="1"/>
-      <cylinder_inertia m="1" r="0.05" h="0.04"/>
-      <inertia
-        ixx="1.0" ixy="0.0" ixz="0.0"
-        iyy="1.0" iyz="0.0"
-        izz="1.0"/>
+        <geometry>
+          <mesh filename="package://mybot_description/meshes/front_wheel.stl" />
+        </geometry>
+    </visual>
+    <inertial>
+        <origin xyz="0 0 0.0" rpy="0 1.5707 1.5707"/>
+        <mass value="1"/>
+        <cylinder_inertia m="1" r="0.05" h="0.04"/>
+        <inertia
+          ixx="1.0" ixy="0.0" ixz="0.0"
+          iyy="1.0" iyz="0.0"
+          izz="1.0"/>
     </inertial>
   </link>
@@ -188,8 +188,14 @@
     <parent link="chassis"/>
     <axis xyz="0 0 0" />
- <joint name="laser_joint" type="fixed">
+  </joint>
+  <joint name="laser_joint" type="fixed">
     <origin xyz="0.17 0 0.1" rpy="0 0 3.1416" />
     <parent link="chassis" />
     <child link="laser" />
+  </joint>
+  <joint name="gps_joint" type="fixed">
+    <origin xyz="0 0.5 0.07"/>
+    <parent link="chassis"/>
+    <child link="gps_link"/>
   </joint>
 <!--
@@ -200,8 +206,3 @@
   </joint>
 -->
-  <joint name="gps_joint" type="fixed">
-    <origin xyz="0 0.5 0.07"/>
-    <parent link="chassis"/>
-    <child link="gps_link"/>
-  </joint>
 </robot>

Commit message: can now import gps_control into other packages

File: simulation/mybot_description/urdf/mybot.xacro (robot description, xacro)
@@ -138,7 +138,7 @@
     </collision>
     <visual name="cam_vis">
-      <origin xyz="0 0 0.028" rpy="0 0 -1.5707"/>
-      <geometry>
-        <mesh filename="package://mybot_description/meshes/sport_camera.dae"/>
+      <origin xyz="0 0 0" rpy="0 0 -1.5707"/>
+      <geometry>
+        <box size="0.05 0.05 0.05"/>
       </geometry>
     </visual>
@@ -184,5 +184,5 @@
   <!-- Sensor joints -->
   <joint type="fixed" name="cam_joint">
-    <origin xyz="0 -0.10 0.07" rpy="0 0 -1.5707"/>
+    <origin xyz="0 -0.10 0.1" rpy="0 0 -1.5707"/>
     <child link="cam_link"/>
     <parent link="chassis"/>

Commit message: shaheer update

File: simulation/mybot_description/urdf/mybot.xacro (robot description, xacro)
@@ -19,6 +19,6 @@
              izz="0.013549"/>
       </inertial>
-    <collision name='collision'>
-      <origin xyz="0.0 0.0 0.0" rpy=" 0 0 0"/>
+    <collision name='collision_chassis'>
+<origin xyz="0.0 0.0 0.0" rpy=" 0 0 0"/>
       <geometry>
         <box size=".4 .2 .1"/>
@@ -26,5 +26,5 @@
     </collision>
     <visual name='chassis_visual'>
-        <origin xyz="0 0 0.06" rpy="0.0 0.0 -1.57" />
+          <origin xyz="0 0 0.06" rpy="0.0 0.0 -1.57" />
         <geometry>
           <mesh filename="package://mybot_description/meshes/frobit_base.stl" />
@@ -54,34 +54,34 @@
     </visual>-->
   </link>
-  <joint name="caster_joint" type="fixed">
-    <parent link="chassis"/>
-    <child link="caster_link"/>
-  </joint>
-  <link name="caster_link">
-    <collision name="collision">
+<joint name="caster_joint" type="fixed">
+            <parent link="chassis"/>
+            <child link="caster_link"/>
+      </joint>
+<link name="caster_link">
+    <collision name="collision_caster">
       <origin xyz="0.15 0 0.06" rpy=" 0 0 0"/>
-        <geometry>
-          <cylinder radius="0.05" length="0.04"/>
-        </geometry>
+      <geometry>
+        <cylinder radius="0.05" length="0.04"/>
+      </geometry>
     </collision>
     <visual name="caster_visual">
       <origin xyz="0.15 0 0.06" rpy=" 0 0 -1.57"/>
-        <geometry>
-          <mesh filename="package://mybot_description/meshes/front_wheel.stl" />
-        </geometry>
-    </visual>
-    <inertial>
-        <origin xyz="0 0 0.0" rpy="0 1.5707 1.5707"/>
-        <mass value="1"/>
-        <cylinder_inertia m="1" r="0.05" h="0.04"/>
-        <inertia
-          ixx="1.0" ixy="0.0" ixz="0.0"
-          iyy="1.0" iyz="0.0"
-          izz="1.0"/>
+      <geometry>
+        <mesh filename="package://mybot_description/meshes/front_wheel.stl" />
+      </geometry>
+    </visual>
+<inertial>
+      <origin xyz="0 0 0.0" rpy="0 1.5707 1.5707"/>
+      <mass value="1"/>
+      <cylinder_inertia m="1" r="0.05" h="0.04"/>
+      <inertia
+        ixx="1.0" ixy="0.0" ixz="0.0"
+        iyy="1.0" iyz="0.0"
+        izz="1.0"/>
     </inertial>
   </link>
   <link name="left_wheel">
     <!--origin xyz="0.1 0.13 0.1" rpy="0 1.5707 1.5707"/-->
-    <collision name="collision">
+    <collision name="collision_left_wheel">
       <origin xyz="0 0 0.0" rpy="0 1.5707 1.5707"/>
       <geometry>
@@ -107,5 +107,5 @@
   <link name="right_wheel">
     <!--origin xyz="0.1 -0.13 0.1" rpy="0 1.5707 1.5707"/-->
-    <collision name="collision">
+    <collision name="collision_right_wheel">
       <origin xyz="0 0 0.0" rpy="0 1.5707 1.5707"/>
       <geometry>
@@ -129,41 +129,4 @@
     </inertial>
   </link>
-   <!-- Sensor links -->
-  <link name="cam_link">
-    <collision name="cam_collision">
-      <origin xyz="0 0 0" rpy="0 0 0"/>
-      <geometry>
-        <box size="0.05 0.05 0.05"/>
-      </geometry>
-    </collision>
-    <visual name="cam_vis">
-      <origin xyz="0 0 0" rpy="0 0 -1.5707"/>
-      <geometry>
-        <box size="0.05 0.05 0.05"/>
-      </geometry>
-    </visual>
-  </link>
-  <link name="laser">
-    <visual>
-      <geometry>
-        <mesh filename="package://mybot_description/meshes/hokuyo.dae" />
-      </geometry>
-      <material name="Green"/>
-    </visual>
-  </link>
-  <link name="gps_link">
-    <visual>
-      <origin xyz="0 0 0" rpy="0 0 0" />
-      <geometry>
-        <box size="0.01 0.01 0.01" />
-      </geometry>
-    </visual>
-    <collision>
-      <origin xyz="0 0 0" rpy="0 0 0" />
-      <geometry>
-        <box size="0.01 0.01 0.01" />
-      </geometry>
-    </collision>
-  </link>
   <joint type="continuous" name="left_wheel_hinge">
     <origin xyz="-0.07 0.09 0" rpy="0 0 0"/>
@@ -182,20 +145,8 @@
     <joint_properties damping="1.0" friction="0.1"/>
   </joint>
-  <!-- Sensor joints -->
-  <joint type="fixed" name="cam_joint">
-    <origin xyz="0 -0.10 0.1" rpy="0 0 -1.5707"/>
-    <child link="cam_link"/>
-    <parent link="chassis"/>
-    <axis xyz="0 0 0" />
-  </joint>
-  <joint name="laser_joint" type="fixed">
-    <origin xyz="0.17 0 0.1" rpy="0 0 3.1416" />
+ <joint name="laser_joint" type="fixed">
+    <origin xyz="0.17 0 0.15" rpy="0 0 0" />
     <parent link="chassis" />
     <child link="laser" />
-  </joint>
-  <joint name="gps_joint" type="fixed">
-    <origin xyz="0 0.5 0.07"/>
-    <parent link="chassis"/>
-    <child link="gps_link"/>
   </joint>
 <!--
@@ -206,3 +157,65 @@
   </joint>
 -->
+<link name="cam_link">
+    <collision name="cam_collision">
+      <origin xyz="0 0 0" rpy="0 0 0"/>
+      <geometry>
+        <box size="0.05 0.05 0.05"/>
+      </geometry>
+    </collision>
+    <visual name="cam_vis">
+      <origin xyz="0 0 0" rpy="0 0 -1.5707"/>
+      <geometry>
+        <box size="0.05 0.05 0.05"/>
+      </geometry>
+    </visual>
+  </link>
+<joint type="fixed" name="cam_joint">
+    <origin xyz="0 -0.10 0.1" rpy="0 0 -1.5707"/>
+    <child link="cam_link"/>
+    <parent link="chassis"/>
+    <axis xyz="0 0 0" />
+  </joint>
+<link name="gps_link">
+    <visual>
+      <origin xyz="0 0 0" rpy="0 0 0" />
+      <geometry>
+        <box size="0.01 0.01 0.01" />
+      </geometry>
+    </visual>
+    <collision>
+      <origin xyz="0 0 0" rpy="0 0 0" />
+      <geometry>
+        <box size="0.01 0.01 0.01" />
+      </geometry>
+    </collision>
+  </link>
+ <joint name="gps_joint" type="fixed">
+    <origin xyz="0 0 0.085"/>
+    <parent link="chassis"/>
+    <child link="gps_link"/>
+  </joint>
+<link name="laser">
+     <collision name="collision_right_wheel">
+      <origin xyz="0 0 -0.04" rpy="0 0 0"/>
+      <geometry>
+        <mesh filename="package://mybot_description/meshes/hokuyo.dae" />
+      </geometry>
+    </collision>
+	<visual>
+<origin xyz="0 0 -0.04" rpy="0 0 0"/>
+	<geometry>
+	<mesh filename="package://mybot_description/meshes/hokuyo.dae" />
+ 	</geometry>
+	<material name="Green"/>
+	</visual>
+	<inertial>
+<origin xyz="0 0 -0.035 " rpy="0 0 0"/>
+ 	<mass value="0.001"/>
+	<inertia
+	ixx="0.0001" ixy="0.0" ixz="0.0"
+	iyy="0.0001" iyz="0.0"
+ 	izz="0.0001"/>
+ 	</inertial>
+ </link>
 </robot>

Commit message: added frobit which can drive and turn somewhat properly

File: simulation/mybot_description/urdf/mybot.xacro (robot description, xacro)
@@ -62,5 +62,5 @@
       <origin xyz="0.15 0 0.06" rpy=" 0 0 0"/>
       <geometry>
-        <cylinder radius="0.05" length="0.04"/>
+        <cylinder radius="0.05" length="0.04"/> <!--USE SPHERE IF NOT LAGGING WHEN TURNING-->
       </geometry>
     </collision>
